Commit message: runnable for hercules

File: ros/hercules_description/urdf/accessories/kinect_camera.urdf.xacro (robot description, xacro)
@@ -34,5 +34,5 @@
         <origin xyz="0 0 0" rpy="0 0 ${M_PI/2}"/>
         <geometry>
-          <mesh filename="package://husky_description/meshes/accessories/kinect.dae" />
+          <mesh filename="package://hercules_description/meshes/accessories/kinect.dae" />
         </geometry>
       </visual>

File: ros/hercules_description/urdf/accessories/sensor_arch.urdf.xacro (robot description, xacro)
@@ -7,5 +7,5 @@
              <visual>
                  <geometry>
-                     <mesh filename="package://husky_description/meshes/accessories/${size}_mm_sensor_arch.dae" />
+                     <mesh filename="package://hercules_description/meshes/accessories/${size}_mm_sensor_arch.dae" />
                  </geometry>
              </visual>
@@ -13,5 +13,5 @@
                  <origin xyz="0 0 0" rpy="0 0 0"/>
                  <geometry>
-                     <mesh filename="package://husky_description/meshes/accessories/${size}_mm_sensor_arch.dae" />
+                     <mesh filename="package://hercules_description/meshes/accessories/${size}_mm_sensor_arch.dae" />
                  </geometry>
              </collision>

File: ros/hercules_description/urdf/accessories/sick_lms100.urdf.xacro (robot description, xacro)
@@ -42,5 +42,5 @@
         <origin xyz="0 0 0" rpy="0 0 0" />
         <geometry>
-          <mesh filename="package://husky_description/meshes/accessories/sick_lms100.dae" />
+          <mesh filename="package://hercules_description/meshes/accessories/sick_lms100.dae" />
         </geometry>
       </visual>

File: ros/hercules_description/urdf/decorations.urdf.xacro (robot description, xacro)
@@ -21,6 +21,6 @@
 ARISING IN ANY WAY OUT OF THE USE OF THIS SOFTWARE, EVEN IF ADVISED OF THE POSSIBILITY OF SUCH DAMAGE.
 -->
-<robot name="husky_decorations" xmlns:xacro="http://ros.org/wiki/xacro">
-  <xacro:macro name="husky_decorate">
+<robot name="hercules_decorations" xmlns:xacro="http://ros.org/wiki/xacro">
+  <xacro:macro name="hercules_decorate">
     <!-- Spawn Husky chassis -->
     <link name="top_chassis_link">
@@ -28,5 +28,5 @@
         <origin xyz="0 0 0" rpy="0 0 0" />
         <geometry>
-          <mesh filename="package://husky_description/meshes/top_chassis.dae" />
+          <mesh filename="package://hercules_description/meshes/top_chassis.dae" />
         </geometry>
       </visual>
@@ -41,5 +41,5 @@
       <visual>
         <geometry>
-          <mesh filename="package://husky_description/meshes/user_rail.dae" />
+          <mesh filename="package://hercules_description/meshes/user_rail.dae" />
         </geometry>
       </visual>
@@ -55,5 +55,5 @@
       <visual>
         <geometry>
-          <mesh filename="package://husky_description/meshes/bumper.dae" />
+          <mesh filename="package://hercules_description/meshes/bumper.dae" />
         </geometry>
       </visual>
@@ -69,5 +69,5 @@
       <visual>
         <geometry>
-          <mesh filename="package://husky_description/meshes/bumper.dae" />
+          <mesh filename="package://hercules_description/meshes/bumper.dae" />
         </geometry>
       </visual>
@@ -84,5 +84,5 @@
         <origin xyz="0 0 0" rpy="0 0 0" />
         <geometry>
-          <mesh filename="package://husky_description/meshes/top_plate.dae" />
+          <mesh filename="package://hercules_description/meshes/top_plate.dae" />
         </geometry>
       </visual>
@@ -90,5 +90,5 @@
         <origin xyz="0 0 0" rpy="0 0 0"/>
         <geometry>
-          <mesh filename="package://husky_description/meshes/top_plate.dae" />
+          <mesh filename="package://hercules_description/meshes/top_plate.dae" />
         </geometry>
       </collision>

File: ros/hercules_description/urdf/hercules.urdf.xacro (robot description, xacro)
@@ -106,5 +106,5 @@
       <origin xyz="${-wheelbase/2} ${-track/2} ${wheel_vertical_offset}" rpy="0 0 0" />
     </xacro:hercules_wheel>
-    <xacro:husky_decorate />
+    <xacro:hercules_decorate />
     <xacro:if value="$(arg ur5_enabled)">
       <xacro:property name="reflect" value="-1" />

File: ros/hercules_description/urdf/wheel.urdf.xacro (robot description, xacro)
@@ -32,5 +32,5 @@
 				<origin xyz="0 0 0" rpy="0 0 0" />
 				<geometry>
-					<mesh filename="package://husky_description/meshes/wheel.dae" />
+					<mesh filename="package://hercules_description/meshes/wheel.dae" />
 				</geometry>
 			</visual>
